File: ESP32/Easyduino_ESP32.kicad_pcb (KiCad board)
At the start: 4 copper layers, 28.4 x 47.9 mm, 27 parts, among them J1 USB_C_Receptacle_USB2.0, Q1 SS8050, Q2 SS8050, SW1 SW_Push, SW2 SW_Push, U1 CP2102N-Axx-xQFN28, U2 ESP32-WROOM-E, U3 AMS1117-3.3, U4 ESP32-DevKitC

Commit message: ESP32 CP2102 bugfix
Parts:
- added R7: 10k, Resistor_SMD:R_0402_1005Metric, F.Cu at (150.3, 101.3)
- added R8: 5.1k, Resistor_SMD:R_0402_1005Metric, F.Cu at (150.3, 102.3)
Connections:
- net +5V renamed VBUS
- U1 pad 11: unconnected-(U1-~{SUSPEND}-Pad11) -> /~{SUSPEND}
- U1 pad 9: GND -> /~{RST}
Routing:
- net /~{SUSPEND}: track 0.00 -> 1.78 mm
- net /~{RST}: track 0.00 -> 1.78 mm
- net VBUS: track 57.2 -> 56.5 mm
- net GND: track 36.0 -> 35.9 mm, vias 30 -> 31
Other:
- board text added: "Designed with KiCad v10 https://github.com/Hanqaqa/Easyduino"
- board text removed: "Designed with KiCad v7 https://github.com/Hanqaqa/Easyduino"
