File: Raspberry Pi Pico 2040/Easyduino_RP2040.kicad_sch (KiCad schematic)
At the start: 66 parts, among them J1 USB_C_Receptacle_USB2.0, J3 Conn_01x20, J4 Conn_01x20, J5 Conn_01x03, J6 Conn_01x03_MountingPin, J7 Conn_01x01_Pin, SW1 SW_Push, SW2 SW_Push, U1 XC6206P332MR, U2 RP2040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

Commit message: RP2040 v1.2
Parts:
- removed J7: Conn_01x01_Pin, Connector_PinHeader_2.54mm:PinHeader_1x01_P2.54mm_Vertical, symbol Connector:Conn_01x01_Pin
- R10, R11, R8: now left out of the parts list
Connections:
- net SWCLK: now also J6.1 (Pin_1); no longer J6.3 (Pin_3)
- net SWD: now also J6.3 (Pin_3); no longer J6.1 (Pin_1)
Other:
- note added: "BootSel"
- note added: "Reset"
Changed lines of the file:
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@@
 		)
 	)
+	(text "BootSel"
+		(exclude_from_sim no)
+		(at 23.622 215.138 0)
+		(effects
+			(font
+				(size 1.27 1.27)
+				(thickness 0.8)
+				(bold yes)
+			)
+			(justify left bottom)
+		)
+	)
 	(text "Both 1uF caps close to the regulator"
 		(exclude_from_sim no)
@@
 		)
 	)
+	(text "Reset"
+		(exclude_from_sim no)
+		(at 48.514 215.138 0)
+		(effects
+			(font
+				(size 1.27 1.27)
+				(thickness 0.8)
+				(bold yes)
+			)
+			(justify left bottom)
+		)
+	)
 	(text "USB"
 		(exclude_from_sim no)
@@
 	(wire
 		(pts
-			(xy 57.15 243.84) (xy 50.8 243.84)
+			(xy 59.69 243.84) (xy 50.8 243.84)
 		)
 		(stroke
@@
 	)
 	(label "RUN"
-		(at 52.07 243.84 0)
+		(at 59.69 243.84 180)
 		(fields_autoplaced yes)
 		(effects
@@
 				(size 1.27 1.27)
 			)
-			(justify left bottom)
+			(justify right bottom)
 		)
 		(property "Sheet References" ""
-			(at 52.07 245.11 0)
+			(at 59.69 245.11 0)
 			(hide yes)
 			(show_name no)
@@
 					(size 1.27 1.27)
 				)
-				(justify left)
+				(justify right)
 			)
 		)
@@
 		)
 	)
-	(label "SWD"
-		(at 148.59 180.34 180)
-		(fields_autoplaced yes)
-		(effects
-			(font
-				(size 1.27 1.27)
-			)
-			(justify right bottom)
-		)
-		(property "Sheet References" ""
-			(at 148.59 181.61 0)
-			(hide yes)
-			(show_name no)
-			(do_not_autoplace no)
-			(effects
-				(font
-					(size 1.27 1.27)
-				)
-				(justify right)
-			)
-		)
-	)
 	(label "GPIO12"
 		(at 342.9 91.44 180)
@@
 		)
 	)
-	(label "SWCLK"
-		(at 148.59 185.42 180)
-		(fields_autoplaced yes)
+	(label "GPIO11"
+		(at 342.9 88.9 180)
 		(effects
 			(font
@@
 			(justify right bottom)
 		)
-		(property "Sheet References" ""
-			(at 148.59 186.69 0)
-			(hide yes)
-			(show_name no)
-			(do_not_autoplace no)
-			(effects
-				(font
-					(size 1.27 1.27)
-				)
-				(justify right)
-			)
-		)
 	)
-	(label "GPIO11"
-		(at 342.9 88.9 180)
+	(label "SWD"
+		(at 148.59 185.42 180)
 		(effects
 			(font
@@
 		)
 	)
+	(label "SWCLK"
+		(at 148.59 180.34 180)
+		(effects
+			(font
+				(size 1.27 1.27)
+			)
+			(justify right bottom)
+		)
+	)
 	(label "GPIO0"
 		(at 342.9 60.96 180)
@@
 	)
 	(symbol
-		(lib_id "Connector:Conn_01x01_Pin")
-		(at 62.23 243.84 180)
-		(unit 1)
-		(body_style 1)
-		(exclude_from_sim no)
-		(in_bom yes)
-		(on_board yes)
-		(in_pos_files yes)
-		(dnp no)
-		(property "Reference" "J7"
-			(at 58.166 240.538 0)
-			(show_name no)
-			(do_not_autoplace no)
-			(effects
-				(font
-					(size 1.27 1.27)
-				)
-			)
-		)
-		(property "Value" "Conn_01x01_Pin"
-			(at 61.595 246.38 0)
-			(hide yes)
-			(show_name no)
-			(do_not_autoplace no)
-			(effects
-				(font
-					(size 1.27 1.27)
-				)
-			)
-		)
-		(property "Footprint" "Connector_PinHeader_2.54mm:PinHeader_1x01_P2.54mm_Vertical"
-			(at 62.23 243.84 0)
-			(hide yes)
-			(show_name no)
-			(do_not_autoplace no)
-			(effects
-				(font
-					(size 1.27 1.27)
-				)
-			)
-		)
-		(property "Datasheet" ""
-			(at 62.23 243.84 0)
-			(hide yes)
-			(show_name no)
-			(do_not_autoplace no)
-			(effects
-				(font
-					(size 1.27 1.27)
-				)
-			)
-		)
-		(property "Description" "Generic connector, single row, 01x01, script generated"
-			(at 62.23 243.84 0)
-			(hide yes)
-			(show_name no)
-			(do_not_autoplace no)
-			(effects
-				(font
-					(size 1.27 1.27)
-				)
-			)
-		)
-		(pin "1"
-		)
-		(instances
-			(project "Easyduino_RP2040"
-				(path "/9eec604e-4498-4c8d-831f-8e3bb6ce48eb"
-					(reference "J7")
-					(unit 1)
-				)
-			)
-		)
-	)
-	(symbol
 		(lib_id "Device:R")
 		(at 260.35 116.84 90)
@@
 		(body_style 1)
 		(exclude_from_sim no)
-		(in_bom yes)
+		(in_bom no)
 		(on_board yes)
 		(in_pos_files yes)
@@
 		(body_style 1)
 		(exclude_from_sim no)
-		(in_bom yes)
+		(in_bom no)
 		(on_board yes)
 		(in_pos_files yes)
@@
 		(body_style 1)
 		(exclude_from_sim no)
-		(in_bom yes)
+		(in_bom no)
 		(on_board yes)
 		(in_pos_files yes)
