File: Raspberry Pi Pico 2040/Easyduino_RP2040.kicad_pcb (KiCad board)
At the start: 4 copper layers, 21 x 51 mm, 66 parts, among them J1 USB_C_Receptacle_USB2.0, J3 Conn_01x20, J4 Conn_01x20, J5 Conn_01x03, J6 Conn_01x03_MountingPin, J7 Conn_01x01_Pin, SW1 SW_Push, SW2 SW_Push, U1 XC6206P332MR, U2 RP2040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

Commit message: RP2040 v1.2
Parts:
- removed J7: Conn_01x01_Pin, Connector_PinHeader_2.54mm:PinHeader_1x01_P2.54mm_Vertical
- moved J6 0.10 mm to (144.5, 118.2), turned to 0 degrees
Connections:
- J6 pad 1: /SWD -> /SWCLK
- J6 pad 3: /SWCLK -> /SWD
Routing:
- net /RUN: vias 1 -> 2
Other:
- board text added: "BT"
- board text added: "RST"

Commit message: RP2040 v1.2 SilkScreen Fix
Other:
- board text removed: "V1.1.1"
Changed lines of the file:
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@@
-		)
-	)
-	(gr_text "V1.1.1"
-		(at 147.11 77.17 0)
-		(layer "B.SilkS")
-		(effects
-			(font
-				(size 1 1)
-				(thickness 0.15)
-			)
-			(justify left bottom mirror)
 		)
 	)
